Commit message: Minoir changes

File: src/kuka_description/urdf/gripper.xacro (robot description, xacro)
@@ -91,7 +91,7 @@
             <child link="${prefix}gripper_right_finger_link" />
             <origin xyz="0.07 0 0.02" rpy="0 0 0" />
-            <axis xyz="-1 0 0" />
-            <limit effort="100.0" velocity="0.5" lower="0.0" upper="0.06" />
-            <mimic joint="${prefix}gripper_left_finger_joint" multiplier="1.0" offset="0.0"/>
+            <axis xyz="1 0 0" />
+            <limit effort="100.0" velocity="0.5" lower="-0.06" upper="0.0" />
+            <mimic joint="${prefix}gripper_left_finger_joint" multiplier="-1.0" offset="0.0"/>
         </joint>
         <!-- Gazebo-specific configurations -->

File: src/kuka_description/urdf/kuka_ros2_control.xacro (robot description, xacro)
@@ -66,11 +66,6 @@
         </joint>
         <joint name="gripper_right_finger_joint">
-            <command_interface name="position">
-            <param name="min">0.0</param>
-            <param name="max">0.06</param>
-            </command_interface>
-            <state_interface name="position"/>
             <param name="mimic">gripper_left_finger_joint</param>
-            <param name="multiplier">1.0</param>
+            <param name="multiplier">-1.0</param>
         </joint>
     </ros2_control>
