Commit message: Added a simple gripper

File: src/kuka_description/urdf/kr10r1420.urdf.xacro (robot description, xacro)
@@ -2,4 +2,5 @@
 <robot xmlns:xacro="http://www.ros.org/wiki/xacro" name="kuka_kr10r1420">
   <xacro:include filename="$(find kuka_description)/resources/common_materials.xacro"/>
+  <xacro:include filename="$(find kuka_description)/urdf/gripper.xacro"/>
   <xacro:arg name="is_ignition" default="true"/>
   <xacro:include filename="$(find kuka_description)/urdf/kuka_gazebo.xacro" />
@@ -193,4 +194,8 @@
       <origin xyz="0 0 0" rpy="0 ${radians(90)} 0"/>
     </joint>
+    <!-- Add gripper to the flange -->
+    <xacro:simple_gripper prefix="${prefix}" parent="${prefix}flange">
+      <origin xyz="0 0 0" rpy="0 ${radians(90)} 0"/>
+    </xacro:simple_gripper>
   </xacro:macro>
   <!-- Instantiate the macro once to create the robot -->

File: src/kuka_description/urdf/kuka_ros2_control.xacro (robot description, xacro)
@@ -58,4 +58,20 @@
             <state_interface name="position"/>
         </joint>
+        <joint name="gripper_left_finger_joint">
+            <command_interface name="position">
+            <param name="min">0.0</param>
+            <param name="max">0.06</param>
+            </command_interface>
+            <state_interface name="position"/>
+        </joint>
+        <joint name="gripper_right_finger_joint">
+            <command_interface name="position">
+            <param name="min">0.0</param>
+            <param name="max">0.06</param>
+            </command_interface>
+            <state_interface name="position"/>
+            <param name="mimic">gripper_left_finger_joint</param>
+            <param name="multiplier">1.0</param>
+        </joint>
     </ros2_control>
 </robot>

Commit message: Added camera and 3 RGB boxes

File: src/kuka_description/urdf/kr10r1420.urdf.xacro (robot description, xacro)
@@ -3,4 +3,5 @@
   <xacro:include filename="$(find kuka_description)/resources/common_materials.xacro"/>
   <xacro:include filename="$(find kuka_description)/urdf/gripper.xacro"/>
+  <xacro:include filename="$(find kuka_description)/urdf/camera.xacro"/>
   <xacro:arg name="is_ignition" default="true"/>
   <xacro:include filename="$(find kuka_description)/urdf/kuka_gazebo.xacro" />
@@ -201,3 +202,7 @@
   <!-- Instantiate the macro once to create the robot -->
   <xacro:kuka_kr10r1420 prefix=""/>
+  <!-- Add RGB camera mounted in the world, pointing straight down at boxes -->
+  <xacro:rgb_camera parent="world">
+    <origin xyz="1.0 0.0 1.5" rpy="0 ${pi/2} 0"/>
+  </xacro:rgb_camera>
 </robot>
